File: source/wandfernsprecher/bells.kicad_sch (KiCad schematic)
At the start: 26 parts, among them Q1 AO3400A, Q2 2N5551, Q3 2N5551, Q4 2N5551, Q5 2N5401, Q6 2N5551, Q7 2N5401, Q8 AO3401A, U4 LT1170CT

Commit message: completed layout
Parts:
- C13, C15: value 1µ -> 1µF
- L1: footprint FeWAp:CONN_01x02_vertical -> FeWAp:CONN_01x02_vertical_mod
Connections:
- net at Q4.1 (E), Q5.1 (E): now also L1.1; no longer C15.1
- net at C15.2: now also L1.2; no longer L1.1
- net HV-IN: now reaches C12.1, L2.1, Q8.3 (D), U4.5 (V_{IN})
- net ~{HV_EN}: now reaches Q1.3 (D), R10.1, R9.1
- net HV_{C}': now reaches C13.1, R16.1
- net HV-C: now reaches R16.2, U4.1 (V_{C})
- net at Q6.1 (E), Q7.1 (E): now also C15.1; no longer L1.2
- net HV-FB: now reaches R17.1, R18.2, U4.2 (FB)
Other:
- moved on the sheet: C15, L1

Commit message: cleanup and 3D-Models fixed submodule updated README
Other:
- company: (none) -> author: ${author}
- title: (none) -> ${title}
Changed lines of the file:
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@@
 	(generator_version "8.0")
 	(paper "A4")
+	(title_block
+		(title "${title}")
+		(date "01.11.2024")
+		(rev "${revision}")
+		(company "author: ${author}")
+	)
 	(junction
 		(at 228.6 113.03)
@@
 	(label "HV-IN"
 		(at 102.87 90.17 0)
-		(fields_autoplaced yes)
 		(effects
 			(font
@@
 	(label "~{HV_EN}"
 		(at 74.93 100.33 180)
-		(fields_autoplaced yes)
 		(effects
 			(font
@@
 	(label "HV-FB"
 		(at 125.73 96.52 0)
-		(fields_autoplaced yes)
 		(effects
 			(font
@@
 	(label "HV_{C}'"
 		(at 110.49 106.68 0)
-		(fields_autoplaced yes)
 		(effects
 			(font
@@
 	(label "HV-C"
 		(at 110.49 96.52 90)
-		(fields_autoplaced yes)
 		(effects
 			(font
@@
 		(shape input)
 		(at 55.88 90.17 180)
-		(fields_autoplaced yes)
 		(effects
 			(font
@@
 		(shape input)
 		(at 210.82 129.54 180)
-		(fields_autoplaced yes)
 		(effects
 			(font
@@
 		(shape input)
 		(at 55.88 106.68 180)
-		(fields_autoplaced yes)
 		(effects
 			(font
@@
 		(shape input)
 		(at 46.99 127 180)
-		(fields_autoplaced yes)
 		(effects
 			(font
@@
 		(shape input)
 		(at 210.82 91.44 180)
-		(fields_autoplaced yes)
-		(effects
-			(font
+		(effects
+			(font
