File: source/wandfernsprecher/pwr_supply.kicad_sch (KiCad schematic)
At the start: 14 parts, among them U3 BQ24090DGQ

Commit message: completed layout
Parts:
- added C10: 100nF, Capacitor_SMD:C_0603_1608Metric, symbol Device:C
- added C8: 10µF, Capacitor_SMD:C_0603_1608Metric, symbol Device:C
- added C9: 10nF, Capacitor_SMD:C_0603_1608Metric, symbol Device:C
- added SW3: SW_SPST, Connector_JST:JST_PH_B2B-PH-K_1x02_P2.00mm_Vertical, symbol Switch:SW_SPST
- added U8: TPS73633DBV, Package_TO_SOT_SMD:SOT-23-5, symbol Regulator_Linear:TPS73633DBV
- BT1: Connector (none) -> JST PH 2mm
- C6, C7: footprint (none) -> Capacitor_SMD:C_0603_1608Metric
- D2, D3: footprint (none) -> LED_SMD:LED_0805_2012Metric
- JP1, JP2: footprint (none) -> Jumper:SolderJumper-2_P1.3mm_Open_RoundedPad1.0x1.5mm
- R28, R29, R30, R31, R32, R33: footprint (none) -> Resistor_SMD:R_0603_1608Metric
Connections:
- net +BATT: now also SW3.1 (A)
- net GND: now also C10.2, C8.2, C9.2, U8.2 (GND)
- net VBUS: now also D2.2 (A), D3.2 (A); no longer R32.2, R33.2
- net ISET2: now reaches R30.1, U3.7 (ISET2)
- net at D3.1 (K): now also R33.2; no longer U3.8 (~{CHG})
- net BQ-~{CHG}: now reaches R33.1
- net BQ-~{CHG}: now also U3.8 (~{CHG}); no longer D3.2 (A)
- net ISET: now reaches R28.1, R29.1, U3.2 (ISET)
- net at D2.1 (K): now also R32.2; no longer U3.5 (~{PG})
- net TS: now reaches R31.1, U3.9 (TS)
- net ISET'': now reaches JP2.2 (B), R29.2
- net BQ-~{PG}: now reaches R32.1
- net BQ-~{PG}: now also U3.5 (~{PG}); no longer D2.2 (A)
- net ISET': now reaches JP1.2 (B), R28.2
- new net: C9.1, U8.4 (NR)
- new net +3.3V: C8.1, U8.5 (OUT)
- new net 4.0V: C10.1, SW3.2 (B), U8.1 (IN), U8.3 (EN)
Other:
- note added: "battery"
- note added: "battery charger"
- moved on the sheet: C6, D2, D3, JP1, JP2, R31, R32, R33

Commit message: added ibom added switch holder FreeCAD file added Vin header and ideal diodes, finalized layout
Parts:
- added J2: Vin, Connector_JST:JST_PH_B2B-PH-K_1x02_P2.00mm_Vertical, symbol Connector_Generic:Conn_01x02
- added Q12, Q14: AO3401A, Package_TO_SOT_SMD:SOT-23, symbol Transistor_FET:AO3401A
- added Q13, Q9: BC857BS, Package_TO_SOT_SMD:SOT-363_SC-70-6, symbol Transistor_BJT:BC857BS
- added R24, R25, R27, R34: 10k, Resistor_SMD:R_0603_1608Metric, symbol Device:R
Connections:
- net GND: now also J2.2 (Pin_2), R24.2, R25.2, R27.2, R34.2
- net VBUS: now also Q12.3 (D), Q9.1 (E1); no longer C6.1, D2.2 (A), D3.2 (A), U3.1 (IN)
- new net: Q12.1 (G), Q9.3 (C2), R25.1
- new net: Q9.2 (B1), Q9.5 (B2), Q9.6 (C1), R24.1
- new net: Q13.3 (C2), Q14.1 (G), R34.1
- new net: J2.1 (Pin_1), Q13.1 (E1), Q14.3 (D)
- new net: Q13.2 (B1), Q13.5 (B2), Q13.6 (C1), R27.1
- new net Vin': C6.1, D2.2 (A), D3.2 (A), Q12.2 (S), Q13.4 (E2), Q14.2 (S), Q9.4 (E2), U3.1 (IN)
Other:
- note added: "VBUS ideal diode"
- note added: "Vin ideal diode"
- moved on the sheet: BT1, C10, C6, C7, C8, C9, D2, D3, JP1, JP2, R28, R29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

Commit message: cleanup and 3D-Models fixed submodule updated README
Other:
- company: (none) -> author: ${author}
- title: (none) -> ${title}
Changed lines of the file:
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@@
 	(generator_version "8.0")
 	(paper "A4")
+	(title_block
+		(title "${title}")
+		(date "01.11.2024")
+		(rev "${revision}")
+		(company "author: ${author}")
+	)
 	(junction
 		(at 214.63 92.71)
@@
 	(label "BQ-~{CHG}"
 		(at 118.11 116.84 0)
-		(fields_autoplaced yes)
 		(effects
 			(font
@@
 	(label "+BATT"
 		(at 36.83 100.33 270)
-		(fields_autoplaced yes)
 		(effects
 			(font
@@
 	(label "+BATT"
 		(at 120.65 99.06 90)
-		(fields_autoplaced yes)
 		(effects
 			(font
@@
 	(label "ISET2"
 		(at 83.82 116.84 0)
-		(fields_autoplaced yes)
 		(effects
 			(font
@@
 	(label "ISET'"
 		(at 57.15 121.92 0)
-		(fields_autoplaced yes)
 		(effects
 			(font
@@
 	(label "ISET''"
 		(at 66.04 121.92 0)
-		(fields_autoplaced yes)
 		(effects
 			(font
@@
 	(label "+BATT"
 		(at 182.88 92.71 0)
-		(fields_autoplaced yes)
 		(effects
 			(font
@@
 	(label "Vin'"
 		(at 149.86 88.9 270)
-		(fields_autoplaced yes)
 		(effects
 			(font
@@
 	(label "ISET"
 		(at 83.82 111.76 0)
-		(fields_autoplaced yes)
 		(effects
 			(font
@@
 	(label "TS"
 		(at 119.38 111.76 0)
-		(fields_autoplaced yes)
 		(effects
 			(font
@@
 	(label "BQ-~{PG}"
 		(at 118.11 121.92 0)
-		(fields_autoplaced yes)
 		(effects
 			(font
@@
 	(label "Vin'"
 		(at 90.17 101.6 90)
-		(fields_autoplaced yes)
 		(effects
 			(font
@@
 		(shape output)
 		(at 120.65 90.17 90)
-		(fields_autoplaced yes)
 		(effects
 			(font
@@
 		(shape output)
 		(at 210.82 88.9 90)
-		(fields_autoplaced yes)
 		(effects
 			(font
@@
 		(shape output)
 		(at 264.16 92.71 0)
-		(fields_autoplaced yes)
 		(effects
 			(font
@@
 		(shape input)
 		(at 35.56 34.29 180)
-		(fields_autoplaced yes)
-		(effects
-			(font
+		(effects
+			(font
