File: source/wandfernsprecher/wandfernsprecher.kicad_pcb (KiCad board)
At the start: 4 copper layers, 132.5 x 82 mm, 91 parts, among them J1 Hörer, J2 Vin, J3 Conn_01x04, Q1 AO3400A, Q10 AO3401A, Q11 AO3400A, Q12 AO3401A, Q13 BC857BS, Q14 AO3401A, Q2 2N5551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

Commit message: connected RING interrupt line from GSM to ESP
Parts:
- added Q15: AO3400A, Package_TO_SOT_SMD:SOT-23, F.Cu at (115.8, 106.2)
- added R35: 1k, Resistor_SMD:R_0603_1608Metric, F.Cu at (112.3, 107.2)
- D4: value 5,1V -> 5.1V
Connections:
- net ES1 renamed RING
- net ES2 renamed ES
- ES1 pad 3: Net-(ES1-C) -> unconnected-(ES1-C-Pad3)_1
- R3 pad 2: Net-(ES1-C) -> Net-(Q15-D)
- U1 pad 11: unconnected-(U1-RING-Pad11) -> Net-(U1-RING)
Routing:
- net Net-(U1-RING): track 0.00 -> 58.2 mm
- net Net-(Q15-D): track 0.00 -> 25.3 mm
- net Net-(ES1-C): track 20.9 -> 0.00 mm
- net unconnected-(SW2-NC-Pad4): track 3.96 -> 0.00 mm
- net (no net): track 0.00 -> 3.96 mm
- net Net-(Q15-G): track 0.00 -> 1.68 mm
