File: source/wandfernsprecher/wandfernsprecher.kicad_sch (KiCad schematic)
At the start: 37 parts, among them J1 Hörer, J3 Conn_01x04, Q10 AO3401A, Q11 AO3400A, SW4 BOOT, U1 SIM800L, U2 ESP32-C3-WROOM-02, U5 USBLC6-2SC6

Commit message: connected RING interrupt line from GSM to ESP
Parts:
- added Q15: AO3400A, Package_TO_SOT_SMD:SOT-23, symbol Transistor_FET:AO3400A
- added R35: 1k, Resistor_SMD:R_0603_1608Metric, symbol Device:R
Connections:
- net GND: now also Q15.2 (S)
- net at R3.2: now also Q15.3 (D); no longer ES1.3 (C)
- net at U1.11 (RING): now also R35.1
- net ES1 renamed RING
- net ES2 renamed ES
- new net: Q15.1 (G), R35.2
Other:
- moved on the sheet: C3, C4, R3
